File: Hassium8K.kicad_pcb (KiCad board)
At the start: 2 copper layers, 59.9 x 63 mm, 52 parts, among them J1 Conn_01x04_Pin, J2 Conn_01x04_Pin, J3 Conn_01x04_Pin, J4 Conn_01x04_Pin, J5 C596731, J6 C596731, J7 Conn_01x08_Pin, SW1 SW_DPST_x2, SW2 SW_DPST_x2, SW3 SW_DPST_x2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

Commit message: Add files via upload
Parts:
- moved C25 0.22 mm to (563.4, 434.0)
Connections:
- U4 pad 10: unconnected-(U4-PA0-Pad10) -> COL7-1
- U4 pad 22: COL7-1 -> unconnected-(U4-PB11-Pad22)
Routing:
- net COL7-1: track 160.6 -> 166.2 mm
- net GND: track 31.1 -> 33.5 mm, vias 55 -> 56
- net COL8-1: track 164.3 -> 163.8 mm
