File: Hassium8K.kicad_sch (KiCad schematic)
At the start: 52 parts, among them J1 Conn_01x04_Pin, J2 Conn_01x04_Pin, J3 Conn_01x04_Pin, J4 Conn_01x04_Pin, J5 C596731, J6 C596731, J7 Conn_01x08_Pin, SW1 SW_DPST_x2, SW2 SW_DPST_x2, SW3 SW_DPST_x2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

Commit message: Add files via upload
Connections:
- net COL7-1: now also U4.10 (PA0); no longer U4.22 (PB11)
